File: Power Hardware V2.0 (live)/Custom Inverter PCB/Half_Bridges.kicad_sch (KiCad schematic)
At the start: 27 parts, among them Q1 CSD19532Q5B, Q2 CSD19532Q5B, Q3 CSD19532Q5B, Q4 CSD19532Q5B, Q5 CSD19532Q5B, Q6 CSD19532Q5B

Commit message: GERBERS
Parts:
- Q1: footprint (none) -> CSD19532Q5B:TRANS_CSD19532Q5B
Changed lines of the file:
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@@
 			)
 		)
-		(property "Footprint" ""
+		(property "Footprint" "CSD19532Q5B:TRANS_CSD19532Q5B"
 			(at 55.88 49.53 0)
 			(effects
