File: Power Hardware V2.0 (live)/Custom Inverter PCB/Custom Inverter PCB.kicad_pcb (KiCad board)
At the start: 2 copper layers, 166 x 143 mm, 82 parts, among them J1 1714971, J2 1714971, J3 1714968, J6 1989764, J7 1714971, J8 1714971, K2 1-1393210-3, Q1 CSD19532Q5B, Q2 CSD19532Q5B, Q3 CSD19532Q5B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

Commit message: Fixed con issue with trace interfering with mosftet HVDC connection
Routing:
- net +3.3V: track 463.0 -> 464.4 mm, vias 7 -> 9
Changed lines of the file:
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@@
+	)
+	(segment
+		(start 109.5 97)
+		(end 109.5 95.5)
+		(width 1)
+		(layer "F.Cu")
+		(net 1)
+	)
+	(segment
+		(start 112 99.5)
+		(end 109.5 97)
+		(width 1)
+		(layer "F.Cu")
+		(net 1)
 	)
 	(segment
@@
 	)
 	(segment
+		(start 112 99.5)
+		(end 113.7 99.5)
+		(width 0.8)
+		(layer "F.Cu")
+		(net 1)
+	)
+	(segment
+		(start 113.7 99.5)
+		(end 117 96.2)
+		(width 0.8)
+		(layer "F.Cu")
+		(net 1)
+	)
+	(segment
 		(start 82.648 152.892)
 		(end 81.6447 151.8887)
@@
 	)
 	(segment
-		(start 88.08 104.128)
-		(end 90.624 101.584)
-		(width 1)
+		(start 113.3 54.308)
+		(end 112.692 54.308)
+		(width 0.8)
+		(layer "F.Cu")
+		(net 1)
+	)
+	(segment
+		(start 125.887 57.895)
+		(end 125.8 57.808)
+		(width 0.4)
 		(layer "F.Cu")
 		(net 1)
@@
 	)
 	(segment
-		(start 125.887 57.895)
-		(end 125.8 57.808)
-		(width 0.4)
-		(layer "F.Cu")
-		(net 1)
-	)
-	(segment
-		(start 109.6 88.8)
-		(end 117 96.2)
+		(start 112.692 54.308)
+		(end 110.5 56.5)
 		(width 0.8)
 		(layer "F.Cu")
@@
 	)
 	(segment
+		(start 125.497 96.2)
+		(end 131.289 90.408)
+		(width 0.8)
+		(layer "F.Cu")
+		(net 1)
+	)
+	(segment
 		(start 135.3 32.308)
 		(end 137.425 32.308)
@@
 	)
 	(segment
-		(start 113.3 54.308)
-		(end 109.6 58.008)
-		(width 0.8)
-		(layer "F.Cu")
-		(net 1)
-	)
-	(segment
 		(start 184.6 149.848)
 		(end 184.6 138.512)
@@
 	)
 	(segment
-		(start 109.6 97.492)
-		(end 109.6 88.8)
-		(width 1)
-		(layer "F.Cu")
-		(net 1)
-	)
-	(segment
 		(start 126.8 33.808)
 		(end 126.8 30.462114)
@@
 	)
 	(segment
-		(start 90.624 101.584)
-		(end 105.508 101.584)
-		(width 1)
-		(layer "F.Cu")
-		(net 1)
-	)
-	(segment
 		(start 129.4186 83.2036)
 		(end 131.3 85.085)
@@
 	)
 	(segment
+		(start 105.508 101.584)
+		(end 90.624 101.584)
+		(width 1)
+		(layer "F.Cu")
+		(net 1)
+	)
+	(segment
+		(start 109.5 95.5)
+		(end 109.6 95.6)
+		(width 1)
+		(layer "F.Cu")
+		(net 1)
+	)
+	(segment
 		(start 121.1 149.848)
 		(end 118.056 152.892)
@@
 	)
 	(segment
-		(start 125.497 96.2)
-		(end 131.289 90.408)
-		(width 0.8)
-		(layer "F.Cu")
-		(net 1)
-	)
-	(segment
-		(start 105.508 101.584)
+		(start 109.6 95.6)
 		(end 109.6 97.492)
 		(width 1)
@@
 	)
 	(segment
+		(start 109.6 97.492)
+		(end 105.508 101.584)
+		(width 1)
+		(layer "F.Cu")
+		(net 1)
+	)
+	(segment
+		(start 90.624 101.584)
+		(end 88.08 104.128)
+		(width 1)
+		(layer "F.Cu")
+		(net 1)
+	)
+	(segment
 		(start 131.3 85.085)
 		(end 131.3 90.397)
@@
 	)
 	(segment
-		(start 109.6 58.008)
-		(end 109.6 88.8)
-		(width 0.8)
-		(layer "F.Cu")
-		(net 1)
-	)
-	(segment
 		(start 72.7674 138.668)
 		(end 81.6447 138.668)
@@
 	)
 	(via
+		(at 110.5 56.5)
+		(size 0.6)
+		(drill 0.3)
+		(layers "F.Cu" "B.Cu")
+		(net 1)
+	)
+	(via
+		(at 109.5 95.5)
+		(size 0.6)
+		(drill 0.3)
+		(layers "F.Cu" "B.Cu")
+		(net 1)
+	)
+	(via
 		(at 144.8 52.308)
 		(size 0.57)
@@
 		(layer "B.Cu")
 		(net 1)
+	)
+	(segment
+		(start 110.5 94.5)
+		(end 109.5 95.5)
+		(width 0.8)
+		(layer "B.Cu")
+		(net 1)
+	)
+	(segment
+		(start 110.5 56.5)
+		(end 110.5 94.5)
+		(width 0.8)
+		(layer "B.Cu")
+		(net 1)

Commit message: GERBERS
Other:
- board text added: "2025 CUSTOM INVERTER V2.0 M.Nguyen C.O'Brien D.Posala A.Truong"
- board text removed: "INVERTER HARDWARE V2.0 M.Nguyen C.O'Brien D.Posala A.Truong"
Changed lines of the file:
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@@
 		)
 	)
-	(gr_text "INVERTER HARDWARE V2.0\nM.Nguyen\nC.O'Brien\nD.Posala\nA.Truong"
+	(gr_text "2025 CUSTOM INVERTER V2.0\nM.Nguyen\nC.O'Brien\nD.Posala\nA.Truong"
 		(at 49.8 127.8 90)
 		(layer "F.SilkS")
