File: Power Hardware V3.0 (Live)/Custom Inverter PCB/Custom Inverter PCB.kicad_pcb (KiCad board)
At the start: 2 copper layers, 166 x 143 mm, 82 parts, among them J1 1714971, J2 1714971, J3 1714968, J6 1989764, J7 1714971, J8 1714971, K2 1-1393210-3, Q1 CSD19532Q5B, Q2 CSD19532Q5B, Q3 CSD19532Q5B, Q4 CSD19532Q5B, Q5 CSD19532Q5B, Q6 CSD19532Q5B, U1 DRV8300DIPWR, U2 TLI4971A050T5E0001XUMA1, U3 TLI4971A050T5E0001XUMA1, U4 TLI4971A050T5E0001XUMA1, U5 LAUNCHXL-F280049C, U6 OP292GSZ-REEL

Commit message: PCB V3 changes
-HV outputs and inputs changed to screw terminals for lugs
- Fuses changes to 50A
- ADC pin for temp sense along with the temp sensing circuit
- Added more pins to motor encoder term for temp sense
Parts:
- removed C2: 0.33uF, Capacitor_SMD:C_0805_2012Metric
- removed CR4: LD1085D2M33R, LD1085D2M33R:D2PAK&slash_A_STM
- removed F1, F2, F3, F4: 250V 30A, 0463030_ER:FUSE_0463_LTF-M
- removed J3: 1714968, PHOENIX_1714968:PHOENIX_1714968
- removed J6: 1989764, PHOENIX_1989764:PHOENIX_1989764
- removed Q1, Q2, Q3, Q4, Q5, Q6: CSD19532Q5B, CSD19532Q5B:TRANS_CSD19532Q5B
- removed U2, U3, U4: TLI4971A050T5E0001XUMA1, TLI4971A:IC_TLI4971A050T5UE0001XUMA1
- added C16: 0.33uF, Capacitor_SMD:C_0805_2012Metric, F.Cu at (265.1, 100.3)
- added C17: 0.1uF, Capacitor_SMD:C_0805_2012Metric, F.Cu at (265.1, 103.3)
- added C18: 0.33uF, Capacitor_SMD:C_0805_2012Metric, F.Cu at (265.1, 106.3)
- added CR5: LD1085D2M33R, LD1085D2M33R:D2PAK&slash_A_STM, F.Cu at (250.2, 129.4)
- added F5: 250VAC 50A, 0463030_ER:FUSE_0463_LTF-M, F.Cu at (297.9, 41.7)
- added F6: 250VAC 50A, 0463030_ER:FUSE_0463_LTF-M, F.Cu at (297.9, 46.6)
- added F7: 250VAC 50A, 0463030_ER:FUSE_0463_LTF-M, F.Cu at (297.9, 51.5)
- added F8: 100VDC 50A, 0463030_ER:FUSE_0463_LTF-M, F.Cu at (262.5, 89.8)
- added J11: 1990041, PHOENIX_1990041:PHOENIX_1990041, F.Cu at (244.9, 122.1)
- added J16: 1714971, 1714971:PHOENIX_1714971, F.Cu at (224.3, 123.1)
- added J17: 1714971, 1714971:PHOENIX_1714971, F.Cu at (224.3, 137.1)
- added MP1: 7461383, M5 Screw Term 7461383:WP-SHFU_7461383, F.Cu at (228.0, 44.7)
- added MP2: 7461383, M5 Screw Term 7461383:WP-SHFU_7461383, F.Cu at (228.0, 55.6)
- added MP3: 7461383, M5 Screw Term 7461383:WP-SHFU_7461383, F.Cu at (228.0, 66.5)
- added MP4: 7461383, M5 Screw Term 7461383:WP-SHFU_7461383, F.Cu at (51.6, 26.2)
- added MP5: 7461383, M5 Screw Term 7461383:WP-SHFU_7461383, F.Cu at (46.2, 145.5)
- added R23: ???, Resistor_SMD:R_0805_2012Metric, F.Cu at (275.9, 113.7)
- added U7: L78M05CDT-TR, L78M05CDT_TR:DPAK_STM-M, F.Cu at (260.7, 129.1)
- C3, C4, C5, CR1, CR2, CR3, R1, R2, R3, R4, R6, R7, U1: moved to F.Cu
- J1, J2: value 1714971 -> 1990041; footprint 1714971:PHOENIX_1714971 -> PHOENIX_1990041:PHOENIX_1990041
- moved J1 210.8 mm to (244.9, 108.5), turned to 0 degrees
- moved C28 202.7 mm to (279.8, 83.9), turned to 0 degrees
- moved C1 201.1 mm to (265.1, 97.3), turned to 0 degrees
- moved C6 197.1 mm to (307.2, 41.4)
- moved C7 191.4 mm to (307.2, 45.6)
- moved C8 188.7 mm to (307.2, 49.9)
- moved J2 188.1 mm to (270.1, 108.5), turned to 0 degrees
- moved J8 185.3 mm to (224.3, 109.0), turned to 0 degrees
- moved TP7 184.3 mm to (301.6, 56.0), turned to 0 degrees
- moved C10 178.9 mm to (244.7, 70.1), turned to 0 degrees
- moved K2 178.6 mm to (264.9, 65.4)
- moved C9 178.6 mm to (244.7, 49.5), turned to 0 degrees
- moved TP2 176.9 mm to (293.4, 60.1), turned to 0 degrees
- moved TP3 176.4 mm to (293.4, 64.1), turned to 0 degrees
- moved J7 176.1 mm to (257.8, 86.6)
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Connections:
- C1 pad 1: +3.3V -> +5V
- J1 pad 1: GND -> Fan_Power
- J1 pad 2: +12V to relay -> Fan_Power
- J2 pad 2: /GateDriver&Power Inputs/PVDD -> /Encoder Input/Temp+
- U5 pad J12_4: +5V -> Net-(U5B-+5V0-PadJ12_4)
- U5 pad J13_4: +5V -> Net-(U5B-+5V0-PadJ12_4)
- U5 pad J3_21: +5V -> Net-(U5B-+5V0-PadJ12_4)
- U5 pad J3_23: unconnected-(U5A-ADCINA5-PadJ3_23) -> /Current sense/ISENA
- U5 pad J3_24: unconnected-(U5A-ADCINB0-PadJ3_24) -> /Current sense/ISENB
- U5 pad J3_25: unconnected-(U5A-ADCINC2-PadJ3_25) -> /Current sense/ISENC
- U5 pad J3_26: unconnected-(U5A-ADCINB1-PadJ3_26) -> /Encoder Input/Temp+
- U5 pad J5_41: unconnected-(U5A-J5_+3.3V-PadJ5_41) -> +3.3V
- U5 pad J7_67: /Current sense/ISENA -> unconnected-(U5A-ADCINC3_P4I-PadJ7_67)
- U5 pad J7_68: /Current sense/ISENB -> unconnected-(U5A-ADCINC5_P6I-PadJ7_68)
- U5 pad J7_69: /Current sense/ISENC -> unconnected-(U5A-ADCINA3_P21-PadJ7_69)
- U5 pad JP5_1: +5V -> Net-(U5B-+5V0-PadJ12_4)
- U5 pad JP7_1: +5V -> Net-(U5B-+5V0-PadJ12_4)
Routing:
- net +3.3V: track 488.5 -> 0.00 mm, vias 9 -> 0
- net +12VDC: track 211.0 -> 0.00 mm, vias 46 -> 0
- net +5V: track 192.3 -> 0.00 mm
- net /Current sense/Vref: track 124.1 -> 0.00 mm, vias 4 -> 0
- net /Current sense/ISENC: track 118.3 -> 0.00 mm, vias 2 -> 0
- net /SEN_100V: track 115.2 -> 0.00 mm, vias 3 -> 0
- net /INLA: track 113.0 -> 0.00 mm, vias 2 -> 0
- net /INHA: track 112.6 -> 0.00 mm, vias 2 -> 0
- net /INHB: track 108.0 -> 0.00 mm, vias 2 -> 0
- net /INLC: track 107.8 -> 0.00 mm, vias 2 -> 0
- net /INHC: track 107.8 -> 0.00 mm, vias 2 -> 0
- net /INLB: track 106.0 -> 0.00 mm, vias 2 -> 0
- net /Current sense/ISENB: track 102.0 -> 0.00 mm, vias 2 -> 0
- net /Current sense/ISENA: track 71.5 -> 0.00 mm, vias 1 -> 0
- net Net-(U5A-~{XRS}-PadJ2_16): track 68.4 -> 0.00 mm
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- removed copper zone on F.Cu, net +100VDC
- removed copper zone on B.Cu, net +100VDC to Relay
- removed copper zone on F.Cu, net +100VDC to Relay
- removed copper zone on F.Cu, net +12V to relay
- removed copper zone on B.Cu, net +12VDC
- removed copper zone on F.Cu, net +12VDC
- removed copper zone on F.Cu, net /Current sense/IA-
- removed copper zone on B.Cu, net /Current sense/IB-
- removed copper zone on F.Cu, net /Current sense/IB-
- removed copper zone on B.Cu, net /Current sense/IC-
- removed copper zone on F.Cu, net /Current sense/IC-
- removed copper zone on B.Cu, net /GateDriver&Power Inputs/PVDD
- removed copper zone on F.Cu, net /GateDriver&Power Inputs/PVDD
- removed copper zone on B.Cu, net /MOTA
- removed copper zone on F.Cu, net /MOTA
- removed copper zone on B.Cu, net /MOTB
- removed copper zone on F.Cu, net /MOTB
- removed copper zone on B.Cu, net /MOTC
- removed copper zone on F.Cu, net /MOTC
- removed copper zone on F.Cu, net /SHA
- removed copper zone on F.Cu, net /SHB
- removed copper zone on F.Cu, net /SHC
- removed copper zone on B.Cu, net GND
- removed copper zone on F.Cu, net GND
- removed copper zone on B.Cu, net Net-(J7-Pad1)
Other:
- board text added: "2025 CUSTOM INVERTER V3 M.Nguyen C.O'Brien D.Posala A.Truong"
- board text removed: "12V"
- board text removed: "12V CNTRL"
- board text removed: "2025 CUSTOM INVERTER V2.1 M.Nguyen C.O'Brien D.Posala A.Truong"
- board text removed: "GND"
- board text removed: "RELAY CNTRL"

Commit message: PCB layout
Parts:
- removed C18: 0.33uF, Capacitor_SMD:C_0805_2012Metric
- removed C21, C23: 47nF, Capacitor_SMD:C_0805_2012Metric
- removed CR5: LD1085D2M33R, LD1085D2M33R:D2PAK&slash_A_STM
- removed F5, F6, F7: 250VAC 50A, 0463030_ER:FUSE_0463_LTF-M
- removed F8: 100VDC 50A, 0463030_ER:FUSE_0463_LTF-M
- removed J16, J17: 1714971, 1714971:PHOENIX_1714971
- removed J2: 1990041, PHOENIX_1990041:PHOENIX_1990041
- removed K2: 1-1393210-3, T9AS1D12_12:TE_1-1393210-3
- removed R32, R35, R36: 220R, Resistor_SMD:R_0805_2012Metric
- removed R43: 97.6K, Resistor_SMD:R_0805_2012Metric
- removed R44, R45, R46, R47, R48: 3K, Resistor_SMD:R_0805_2012Metric
- added C19: 0.33uF, Capacitor_SMD:C_0805_2012Metric, F.Cu at (168.5, 139.5)
- added C2: 330 µF, EEV_FK2A331M:CAP_EEVFK2A331M, F.Cu at (61.3, 49.7)
- added C20: 0.33uF, Capacitor_SMD:C_0805_2012Metric, F.Cu at (162.1, 139.9)
- added C25: 0.1uF, Capacitor_SMD:C_0805_2012Metric, F.Cu at (168.5, 128.5)
- added C27: 220nF, Capacitor_SMD:C_0603_1608Metric, B.Cu at (127.9, 130.6)
- added C29: 220nF, Capacitor_SMD:C_0603_1608Metric, F.Cu at (159.3, 63.1)
- added C30: 220nF, Capacitor_SMD:C_0603_1608Metric, F.Cu at (133.3, 57.1)
- added CR4: LD1085D2M33R, LD1085D2M33R:D2PAK&slash_A_STM, F.Cu at (177.1, 134.0)
- added F1: 100VDC 50A, 0463030_ER:FUSE_0463_LTF-M, F.Cu at (57.7, 36.0)
- added F2: 250VAC 50A, 0463030_ER:FUSE_0463_LTF-M, F.Cu at (112.0, 45.4)
- added F3: 250VAC 50A, 0463030_ER:FUSE_0463_LTF-M, F.Cu at (147.0, 44.9)
- added F4: 250VAC 50A, 0463030_ER:FUSE_0463_LTF-M, F.Cu at (177.0, 45.1)
- added J10: 1990041, PHOENIX_1990041:PHOENIX_1990041, F.Cu at (86.8, 158.2)
- added J6: 1990041, PHOENIX_1990041:PHOENIX_1990041, F.Cu at (191.7, 123.5)
- added J9: 1990009, 2P term 1990009:PHOENIX_1990009, F.Cu at (73.1, 158.2)
- added K1: 1-1393210-3, T9AS1D12_12:TE_1-1393210-3, B.Cu at (86.5, 47.3)
- added Q1: IRFB4115PBF, Package_TO_SOT_THT:TO-220-3_Vertical, F.Cu at (112.0, 67.4)
- added Q2: IRFB4115PBF, Package_TO_SOT_THT:TO-220-3_Vertical, F.Cu at (123.5, 67.4)
- added Q3: IRFB4115PBF, Package_TO_SOT_THT:TO-220-3_Vertical, F.Cu at (137.0, 73.9)
- added Q4: IRFB4115PBF, Package_TO_SOT_THT:TO-220-3_Vertical, F.Cu at (148.8, 73.9)
- added Q5: IRFB4115PBF, Package_TO_SOT_THT:TO-220-3_Vertical, F.Cu at (169.0, 73.8)
- added Q6: IRFB4115PBF, Package_TO_SOT_THT:TO-220-3_Vertical, F.Cu at (180.5, 73.7)
- added R19: 220R, Resistor_SMD:R_0805_2012Metric, B.Cu at (133.2, 124.7)
- added R20: 5.36k, Resistor_SMD:R_0805_2012Metric, F.Cu at (128.1, 127.5)
- added R21: 10k, Resistor_SMD:R_0805_2012Metric, F.Cu at (71.1, 118.7)
- added R22: 3K, Resistor_SMD:R_0805_2012Metric, F.Cu at (67.9, 128.1)
- added R24: 10k, Resistor_SMD:R_0805_2012Metric, F.Cu at (67.9, 125.1)
- added R25: 10k, Resistor_SMD:R_0805_2012Metric, F.Cu at (81.6, 126.2)
- added R26: 3K, Resistor_SMD:R_0805_2012Metric, F.Cu at (83.4, 123.1)
- added R27: 10k, Resistor_SMD:R_0805_2012Metric, F.Cu at (81.6, 120.7)
- added R28: 3K, Resistor_SMD:R_0805_2012Metric, F.Cu at (81.6, 129.1)
- added U2: LAUNCHXL-F280049C, LAUNCHXL-F280049C:MODULE_LAUNCHXL-F280049C, B.Cu at (115.3, 113.3)
- added U3: TLI4971A050T5E0001XUMA1, TLI4971A:TLI4971A050T5UE0001XUMA1, F.Cu at (126.0, 57.5)
- added U4: TLI4971A050T5E0001XUMA1, TLI4971A:TLI4971A050T5UE0001XUMA1, F.Cu at (152.0, 63.5)
- C1: value 0.1uF -> 330 µF; footprint Capacitor_SMD:C_0805_2012Metric -> EEV_FK2A331M:CAP_EEVFK2A331M
- C10: value 330 µF -> 220nF; footprint EEV_FK2A331M:CAP_EEVFK2A331M -> Capacitor_SMD:C_0603_1608Metric
- C14: value 220nF -> 47nF; footprint Capacitor_SMD:C_0603_1608Metric -> Capacitor_SMD:C_0805_2012Metric
- C15: value 0.1uF -> 47nF
- C16: value 0.33uF -> 47nF
- C24: value 47nF -> 0.1uF
- C28: value 0.1uF -> 220nF; footprint Capacitor_SMD:C_0805_2012Metric -> Capacitor_SMD:C_0603_1608Metric
- C3: value 1uF -> 0.1uF; moved to B.Cu
- C6: footprint Capacitor_SMD:C_1210_3225Metric -> Capacitor_SMD:C_0805_2012Metric
- C9: value 330 µF -> 1uF; footprint EEV_FK2A331M:CAP_EEVFK2A331M -> Capacitor_SMD:C_1210_3225Metric
- J1: value 1990041 -> 1990009; footprint PHOENIX_1990041:PHOENIX_1990041 -> 2P term 1990009:PHOENIX_1990009
- J8: value 1714971 -> 1990009; footprint 1714971:PHOENIX_1714971 -> 2P term 1990009:PHOENIX_1990009
- R1: value 15R -> 97.6K; moved to B.Cu
- R15, R16: moved to B.Cu
- R17: value 4.7K -> 220R; moved to B.Cu
- R18: value 10k -> 220R; moved to B.Cu
- R2: value 15R -> 3K; moved to B.Cu
- R23: value ??? -> 3K
- R5, R8: value 10k -> 15R
- R9: value 10k -> 4.7K
- U5: value LAUNCHXL-F280049C -> TLI4971A050T5E0001XUMA1; footprint LAUNCHXL-F280049C:MODULE_LAUNCHXL-F280049C -> TLI4971A:TLI4971A050T5UE0001XUMA1; moved to F.Cu
- moved C6 253.0 mm to (60.8, 98.7)
- moved R10 231.0 mm to (69.6, 141.1), turned to 180 degrees
- moved R2 230.6 mm to (61.3, 79.0), turned to 180 degrees
- moved R1 227.3 mm to (65.1, 79.0), turned to 180 degrees
- moved J7 225.6 mm to (43.7, 157.9)
- moved C4 220.6 mm to (60.8, 103.7)
- moved C3 220.2 mm to (66.5, 129.2), turned to 90 degrees
- moved C5 220.0 mm to (60.8, 101.2)
- moved U6 211.7 mm to (75.4, 124.1)
- moved R23 207.1 mm to (69.0, 122.1), turned to -90 degrees
- moved C1 202.9 mm to (63.8, 72.5), turned to 180 degrees
- moved R9 199.5 mm to (73.6, 141.1), turned to 180 degrees
- moved CR1 191.7 mm to (54.9, 103.7), turned to 180 degrees
- moved CR2 191.1 mm to (54.9, 101.2), turned to 180 degrees
- moved CR3 190.8 mm to (54.9, 98.7), turned to 180 degrees
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Connections:
- C1 pad 1: +5V -> +100VDC to Relay
- C10 pad 1: +100VDC to Relay -> /Current sense/Vref
- C12 pad 1: /Current sense/Vref -> GND
- C12 pad 2: GND -> +3.3V
- C14 pad 1: GND -> /Current sense/ISENA
- C14 pad 2: +3.3V -> GND
- C15 pad 1: +5V -> /Current sense/ISENB
- C16 pad 1: +12VDC -> /Current sense/ISENC
- C17 pad 1: +3.3V -> +5V
- C24 pad 1: /Current sense/ISENA -> +5V
- C28 pad 1: /SEN_100V -> /Current sense/Vref
- C3 pad 1: /GateDriver&Power Inputs/CBSTA_HI -> /SEN_100V
- C3 pad 2: /SHA -> GND
- C4 pad 1: /GateDriver&Power Inputs/CBSTB_HI -> /GateDriver&Power Inputs/CBSTA_HI
- C4 pad 2: /SHB -> /SHA
- C5 pad 1: /GateDriver&Power Inputs/CBSTC_HI -> /GateDriver&Power Inputs/CBSTB_HI
- C5 pad 2: /SHC -> /SHB
- C6 pad 1: +100VDC -> /GateDriver&Power Inputs/CBSTC_HI
- C6 pad 2: GND -> /SHC
- C9 pad 1: +100VDC to Relay -> +100VDC
- J1 pad 1: Fan_Power -> Net-(J1-Pad1)
- J1 pad 2: Fan_Power -> +12VDC
- J11 pad 1: GND -> Fan_Power
- J11 pad 3: GND -> Fan_Power
- J11 pad 5: GND -> Fan_Power
- J7 pad 1: Net-(J7-Pad1) -> GND
- J7 pad 2: +12VDC -> +12V to relay
- MP1 pad 1: /MOTA -> /GateDriver&Power Inputs/PVDD
- MP1 pad 10: /MOTA -> /GateDriver&Power Inputs/PVDD
- MP1 pad 11: /MOTA -> /GateDriver&Power Inputs/PVDD
- MP1 pad 12: /MOTA -> /GateDriver&Power Inputs/PVDD
- MP1 pad 13: /MOTA -> /GateDriver&Power Inputs/PVDD
- MP1 pad 14: /MOTA -> /GateDriver&Power Inputs/PVDD
- MP1 pad 15: /MOTA -> /GateDriver&Power Inputs/PVDD
- MP1 pad 16: /MOTA -> /GateDriver&Power Inputs/PVDD
- MP1 pad 2: /MOTA -> /GateDriver&Power Inputs/PVDD
- MP1 pad 3: /MOTA -> /GateDriver&Power Inputs/PVDD
- MP1 pad 4: /MOTA -> /GateDriver&Power Inputs/PVDD
- MP1 pad 5: /MOTA -> /GateDriver&Power Inputs/PVDD
- MP1 pad 6: /MOTA -> /GateDriver&Power Inputs/PVDD
- MP1 pad 7: /MOTA -> /GateDriver&Power Inputs/PVDD
- MP1 pad 8: /MOTA -> /GateDriver&Power Inputs/PVDD
- MP1 pad 9: /MOTA -> /GateDriver&Power Inputs/PVDD
- MP2 pad 1: /MOTB -> GND
- MP2 pad 10: /MOTB -> GND
- MP2 pad 11: /MOTB -> GND
- MP2 pad 12: /MOTB -> GND
- MP2 pad 13: /MOTB -> GND
- MP2 pad 14: /MOTB -> GND
- MP2 pad 15: /MOTB -> GND
- MP2 pad 16: /MOTB -> GND
- MP2 pad 2: /MOTB -> GND
- MP2 pad 3: /MOTB -> GND
- MP2 pad 4: /MOTB -> GND
- MP2 pad 5: /MOTB -> GND
- MP2 pad 6: /MOTB -> GND
- MP2 pad 7: /MOTB -> GND
- MP2 pad 8: /MOTB -> GND
- MP2 pad 9: /MOTB -> GND
- MP3 pad 1: /MOTC -> /MOTA
- MP3 pad 10: /MOTC -> /MOTA
- MP3 pad 11: /MOTC -> /MOTA
- MP3 pad 12: /MOTC -> /MOTA
- MP3 pad 13: /MOTC -> /MOTA
- MP3 pad 14: /MOTC -> /MOTA
- MP3 pad 15: /MOTC -> /MOTA
- MP3 pad 16: /MOTC -> /MOTA
- MP3 pad 2: /MOTC -> /MOTA
- MP3 pad 3: /MOTC -> /MOTA
- MP3 pad 4: /MOTC -> /MOTA
- MP3 pad 5: /MOTC -> /MOTA
- MP3 pad 6: /MOTC -> /MOTA
- MP3 pad 7: /MOTC -> /MOTA
- MP3 pad 8: /MOTC -> /MOTA
- MP3 pad 9: /MOTC -> /MOTA
- MP4 pad 1: /GateDriver&Power Inputs/PVDD -> /MOTB
- MP4 pad 10: /GateDriver&Power Inputs/PVDD -> /MOTB
- MP4 pad 11: /GateDriver&Power Inputs/PVDD -> /MOTB
- MP4 pad 12: /GateDriver&Power Inputs/PVDD -> /MOTB
- MP4 pad 13: /GateDriver&Power Inputs/PVDD -> /MOTB
- MP4 pad 14: /GateDriver&Power Inputs/PVDD -> /MOTB
- MP4 pad 15: /GateDriver&Power Inputs/PVDD -> /MOTB
- MP4 pad 16: /GateDriver&Power Inputs/PVDD -> /MOTB
- MP4 pad 2: /GateDriver&Power Inputs/PVDD -> /MOTB
- MP4 pad 3: /GateDriver&Power Inputs/PVDD -> /MOTB
- MP4 pad 4: /GateDriver&Power Inputs/PVDD -> /MOTB
- MP4 pad 5: /GateDriver&Power Inputs/PVDD -> /MOTB
- MP4 pad 6: /GateDriver&Power Inputs/PVDD -> /MOTB
- MP4 pad 7: /GateDriver&Power Inputs/PVDD -> /MOTB
- MP4 pad 8: /GateDriver&Power Inputs/PVDD -> /MOTB
- MP4 pad 9: /GateDriver&Power Inputs/PVDD -> /MOTB
- MP5 pad 1: GND -> /MOTC
- MP5 pad 10: GND -> /MOTC
- MP5 pad 11: GND -> /MOTC
- MP5 pad 12: GND -> /MOTC
- MP5 pad 13: GND -> /MOTC
- MP5 pad 14: GND -> /MOTC
- MP5 pad 15: GND -> /MOTC
- MP5 pad 16: GND -> /MOTC
- MP5 pad 2: GND -> /MOTC
- MP5 pad 3: GND -> /MOTC
- MP5 pad 4: GND -> /MOTC
- MP5 pad 5: GND -> /MOTC
- MP5 pad 6: GND -> /MOTC
- MP5 pad 7: GND -> /MOTC
- MP5 pad 8: GND -> /MOTC
- MP5 pad 9: GND -> /MOTC
- R1 pad 1: /GateDriver&Power Inputs/GHA -> +100VDC to Relay
- R1 pad 2: Net-(Q1-Pad4) -> /SEN_100V
- R11 pad 2: /Current sense/Vref -> /Current sense/OCD2_A
- R12 pad 2: /Current sense/OCD1_A -> /Current sense/OCD2_B
- R13 pad 2: /Current sense/OCD2_A -> /Current sense/OCD2_C
- R14 pad 2: /Current sense/OCD2_B -> /Current sense/OCD1_A
- R16 pad 2: /Current sense/OCD2_C -> /Current sense/OCD1_C
- R17 pad 1: +3.3V -> /Current sense/1_Out
- R17 pad 2: /Current sense/OCD1_C -> /Current sense/ISENA
- R18 pad 1: +5V -> /Current sense/2_Out
- R18 pad 2: Net-(U6--INB) -> /Current sense/ISENB
- R2 pad 1: /GateDriver&Power Inputs/GLA -> /SEN_100V
- R2 pad 2: Net-(Q2-Pad4) -> GND
- R23 pad 1: /Encoder Input/Temp+ -> /Encoder Input/COS_MCU
- R23 pad 2: +5V -> Net-(U6--INA)
- R3 pad 1: /GateDriver&Power Inputs/GHB -> /GateDriver&Power Inputs/GHA
- R4 pad 1: /GateDriver&Power Inputs/GLB -> /GateDriver&Power Inputs/GLA
- R5 pad 1: Net-(U6-+INA) -> /GateDriver&Power Inputs/GLB
- R5 pad 2: GND -> Net-(Q4-G)
- R6 pad 1: /GateDriver&Power Inputs/GHC -> /GateDriver&Power Inputs/GHB
- R7 pad 1: /GateDriver&Power Inputs/GLC -> /GateDriver&Power Inputs/GHC
- R8 pad 1: +5V -> /GateDriver&Power Inputs/GLC
- R8 pad 2: Net-(U6--INA) -> Net-(Q6-G)
- R9 pad 1: Net-(U6-+INB) -> +3.3V
- R9 pad 2: GND -> /Current sense/Vref
- TP1 pad TP: /MOTA -> /GateDriver&Power Inputs/GHA
- TP2 pad TP: /GateDriver&Power Inputs/GHA -> /GateDriver&Power Inputs/GLA
- TP3 pad TP: /GateDriver&Power Inputs/GHB -> /MOTA
- TP4 pad TP: /GateDriver&Power Inputs/GLA -> /GateDriver&Power Inputs/GHB
Routing:
- net +100VDC to Relay: vias 0 -> 103
- net +100VDC: vias 0 -> 30
- net (no net): vias 4 -> 72
- added copper zone on B.Cu, net +100VDC
- added copper zone on F.Cu, net +100VDC
- added copper zone on B.Cu, net +100VDC to Relay
- added copper zone on F.Cu, net +100VDC to Relay
- added copper zone on B.Cu, net /Current sense/IA-
- added copper zone on F.Cu, net /Current sense/IA-
- added copper zone on B.Cu, net /Current sense/IB-
- added copper zone on F.Cu, net /Current sense/IB-
- added copper zone on B.Cu, net /Current sense/IC-
- added copper zone on F.Cu, net /Current sense/IC-
- added copper zone on F.Cu, net /GateDriver&Power Inputs/PVDD
- added copper zone on B.Cu, net /SHA
- added copper zone on F.Cu, net /SHA
- added copper zone on B.Cu, net /SHB
- added copper zone on F.Cu, net /SHB
- added copper zone on B.Cu, net /SHC
- added copper zone on F.Cu, net /SHC
Other:
- outline, holes or cut-outs redrawn
