File: Power Hardware V3.0 (Live)/Custom Inverter PCB/Custom Inverter PCB.kicad_pcb (KiCad board)
At the start: 2 copper layers, 166 x 143 mm, 93 parts, among them J1 1990009, J10 1990041, J11 1990041, J6 1990041, J7 1714971, J8 1990009, J9 1990009, K1 1-1393210-3, Q1 IRFB4115PBF, Q2 IRFB4115PBF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

Commit message: layout
Parts:
- moved R11 12.6 mm to (127.1, 97.5)
- moved R14 12.5 mm to (130.3, 97.5)
- moved R13 12.4 mm to (139.6, 97.5)
- moved R16 12.2 mm to (142.5, 97.6)
Connections:
- C25 pad 1: +3.3V -> +3.3VDC
- CR4 pad 2: +3.3V -> +3.3VDC
- CR4 pad 4: +3.3V -> +3.3VDC
- R11 pad 1: +3.3V -> +3.3VDC
- R12 pad 1: +3.3V -> +3.3VDC
- R13 pad 1: +3.3V -> +3.3VDC
- R14 pad 1: +3.3V -> +3.3VDC
- R15 pad 1: +3.3V -> +3.3VDC
- R16 pad 1: +3.3V -> +3.3VDC
- R9 pad 1: +3.3V -> +3.3VDC
- U2 pad J11_10: +3.3V -> +3.3VDC
- U2 pad J1_1: +3.3V -> +3.3VDC
- U2 pad J4_37: unconnected-(U2A-GPIO9-PadJ4_37) -> /Current sense/OCD2_B
- U2 pad J4_38: unconnected-(U2A-GPIO8-PadJ4_38) -> /Current sense/OCD1_B
- U2 pad J4_39: unconnected-(U2A-GPIO11-PadJ4_39) -> /Current sense/OCD2_C
- U2 pad J4_40: unconnected-(U2A-GPIO10-PadJ4_40) -> /Current sense/OCD1_C
- U2 pad J5_41: +3.3V -> +3.3VDC
- U2 pad JP4_1: +3.3V -> +3.3VDC
- U2 pad JP6_1: +3.3V -> +3.3VDC
Routing:
- net +3.3VDC: track 0.00 -> 154.8 mm, vias 0 -> 2
- net +3.3V: track 134.2 -> 8.66 mm, vias 1 -> 0
- net /Current sense/OCD2_C: track 0.00 -> 91.2 mm, vias 0 -> 2
- net /Current sense/OCD1_C: track 0.00 -> 90.7 mm
- net /Current sense/OCD2_B: track 19.8 -> 60.9 mm, vias 0 -> 2
- net /Current sense/OCD1_B: track 21.3 -> 59.8 mm, vias 0 -> 2
- net /Current sense/OCD2_A: track 48.2 -> 53.0 mm
- net /Current sense/OCD1_A: track 45.9 -> 50.5 mm
- net GND: track 150.9 -> 148.5 mm
- net /SEN_100V: track 68.2 -> 70.3 mm
- net /Current sense/Vref: track 345.1 -> 343.2 mm, vias 3 -> 4
- net /GateDriver&Power Inputs/GHC: track 117.4 -> 118.8 mm
- net /Current sense/2_Out: track 85.0 -> 86.2 mm
- net /SHC: vias 0 -> 11
- net /SHB: vias 0 -> 13
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
Commit message: V3.0 is ordered
Parts:
- added D10: BRIDGE ON, Capacitor_SMD:C_0603_1608Metric_Pad1.08x0.95mm_HandSolder, F.Cu at (94.7, 79.2)
- added D11: 100V IN, Capacitor_SMD:C_0603_1608Metric_Pad1.08x0.95mm_HandSolder, F.Cu at (80.6, 79.2)
- added D12: 12V, Capacitor_SMD:C_0603_1608Metric_Pad1.08x0.95mm_HandSolder, F.Cu at (49.3, 131.6)
- added D13: 5V, Capacitor_SMD:C_0603_1608Metric_Pad1.08x0.95mm_HandSolder, F.Cu at (153.8, 120.4)
- added D14: 3.3V, Capacitor_SMD:C_0603_1608Metric_Pad1.08x0.95mm_HandSolder, F.Cu at (153.8, 117.1)
- added G***: LOGO, LOGO, F.Cu at (162.9, 90.4)
- added R33: 220R, Resistor_SMD:R_0805_2012Metric, B.Cu at (43.2, 135.9)
- added R34: 220R, Resistor_SMD:R_0805_2012Metric, B.Cu at (47.3, 133.4)
- added R35: 220R, Resistor_SMD:R_0805_2012Metric, F.Cu at (156.7, 121.3)
- added R36: 220R, Resistor_SMD:R_0805_2012Metric, B.Cu at (160.9, 119.7)
- added R37: 220R, Resistor_SMD:R_0805_2012Metric, B.Cu at (161.0, 117.1)
- added R49: 2.7k, Resistor_SMD:R_0805_2012Metric, B.Cu at (96.6, 83.0)
- added R50: 2.7k, Resistor_SMD:R_0805_2012Metric, B.Cu at (94.9, 79.2)
- added R51: 2.7k, Resistor_SMD:R_0805_2012Metric, B.Cu at (76.1, 76.2)
- added R52: 2.7k, Resistor_SMD:R_0805_2012Metric, B.Cu at (76.1, 80.0)
- R4, R5: moved to B.Cu
- moved TP3 19.9 mm to (88.4, 34.8)
- moved TP6 18.4 mm to (124.8, 35.7)
- moved TP9 11.7 mm to (161.2, 36.1)
- moved TP5 5.06 mm to (154.6, 73.5)
- moved R5 4.83 mm to (150.0, 73.2), turned to 180 degrees
- moved C7 3.90 mm to (118.5, 67.1)
- moved C8 3.90 mm to (144.0, 73.6)
- moved C9 3.90 mm to (176.6, 73.4)
- moved Q5 3.90 mm to (169.0, 69.9)
- moved Q6 3.90 mm to (180.5, 69.8)
- moved R3 3.90 mm to (112.0, 67.1)
- moved R6 3.90 mm to (137.0, 73.7)
- moved TP4 3.90 mm to (133.5, 73.6)
- moved TP7 3.90 mm to (163.0, 73.9)
- moved TP8 3.90 mm to (184.5, 74.4)
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Connections:
- C11 pad 2: +3.3V -> +3.3VDC
- C12 pad 2: +3.3V -> +3.3VDC
- C13 pad 2: +3.3V -> +3.3VDC
- U2 pad J12_4: Net-(U2B-+5V0-PadJ12_4) -> unconnected-(U2B-+5V0-PadJ12_4)_3
- U2 pad J13_4: Net-(U2B-+5V0-PadJ12_4) -> unconnected-(U2B-+5V0-PadJ12_4)
- U2 pad J2_16: Net-(U2A-~{XRS}-PadJ2_16) -> unconnected-(U2A-~{XRS}-PadJ2_16)
- U2 pad J3_21: Net-(U2B-+5V0-PadJ12_4) -> unconnected-(U2B-+5V0-PadJ12_4)_2
- U2 pad J6_56: Net-(U2A-~{XRS}-PadJ2_16) -> unconnected-(U2A-~{XRS}-PadJ2_16)_1
- U2 pad JP5_1: Net-(U2B-+5V0-PadJ12_4) -> unconnected-(U2B-+5V0-PadJ12_4)_4
- U2 pad JP7_1: Net-(U2B-+5V0-PadJ12_4) -> unconnected-(U2B-+5V0-PadJ12_4)_1
- U3 pad 1: +3.3V -> +3.3VDC
- U4 pad 1: +3.3V -> +3.3VDC
- U5 pad 1: +3.3V -> +3.3VDC
Routing:
- net +3.3VDC: track 154.8 -> 642.1 mm, vias 2 -> 11
- net /SHC: track 4.14 -> 180.3 mm, vias 11 -> 36
- net /SHB: track 3.90 -> 138.2 mm, vias 13 -> 42
- net +12VDC: track 127.5 -> 251.9 mm, vias 0 -> 3
- net /SHA: track 3.67 -> 120.7 mm, vias 15 -> 50
- net GND: track 148.5 -> 194.0 mm, vias 45 -> 420
- net +12V to relay: track 10.0 -> 30.7 mm
- net /Current sense/Vref: track 343.2 -> 360.7 mm
- net /Current sense/OCD2_A: track 53.0 -> 62.9 mm
- net /Current sense/OCD1_A: track 50.5 -> 60.3 mm, vias 4 -> 2
- net +3.3V: track 8.66 -> 0.00 mm
- net /GateDriver&Power Inputs/GHC: track 118.8 -> 127.4 mm
- net Net-(D14-A): track 0.00 -> 8.06 mm, vias 0 -> 1
- net /Current sense/OCD2_B: track 60.9 -> 68.3 mm, vias 2 -> 1
- net /GateDriver&Power Inputs/GHA: track 77.8 -> 84.7 mm
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- added copper zone on In2.Cu, net +100VDC
- added copper zone on In2.Cu, net +100VDC to Relay
- added copper zone on In2.Cu, net /Current sense/IA-
- added copper zone on In2.Cu, net /Current sense/IB-
- added copper zone on In2.Cu, net /Current sense/IC-
- added copper zone on In2.Cu, net /GateDriver&Power Inputs/PVDD
- added copper zone on In2.Cu, net /MOTA
- added copper zone on In2.Cu, net /MOTB
- added copper zone on In2.Cu, net /MOTC
- added copper zone on In2.Cu, net /SHA
- added copper zone on In2.Cu, net /SHB
- added copper zone on In2.Cu, net /SHC
- added copper zone on B.Cu, net GND
- added copper zone on F.Cu, net GND
- added copper zone on In1.Cu, net GND
Other:
- outline, holes or cut-outs redrawn
- copper layers 2 -> 4
- board text added: "+12V"
- board text added: "+5V | GND | COS | SIN | TMP+ | TMP-"
- board text added: "+B"
- board text added: "- + - + - +"
- board text added: "-B"
- board text added: "100V IN"
- board text added: "100V SWTCH"
- board text added: "12V POWER"
- board text added: "12V SWTCH"
- board text added: "2025 CUSTOM INVERTER V3 (4 Layers) Minh Nguyen David Posala Andy Truong Collin O'Brien"
- board text added: "3.3V ON"
- board text added: "5V ON"
- board text added: "A"
- board text added: "B"
- board text added: "BRIDGE ON"
- board text added: "C"
- board text added: "COOLING FAN OUT"
- board text added: "ENCODER"
- board text added: "FAN CTRL SWTCH"
- board text added: "GND"
- board text removed: "2025 CUSTOM INVERTER V3 M.Nguyen C.O'Brien D.Posala A.Truong"
