File: Power Hardware V3.0 (Live)/Custom Inverter PCB/MCU.kicad_sch (KiCad schematic)
At the start: 5 parts, among them J10 10897202, J4 10897202, J5 10897202, J9 10897202, U5 LAUNCHXL-F280049C

Commit message: Added 100-12 and 12-5 regulators added fan headers
Connections:
- net +5V: no longer U5.J12_4 (+5V0), U5.J13_4 (+5V0), U5.J3_21 (+5V0), U5.JP5_1 (+5V0), U5.JP7_1 (+5V0)
- new net: U5.J12_4 (+5V0), U5.J13_4 (+5V0), U5.J3_21 (+5V0), U5.JP5_1 (+5V0), U5.JP7_1 (+5V0)
- no-connect marks 0 -> 1
Changed lines of the file:
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@@
 		)
+	)
+	(no_connect
+		(at 254 35.56)
 	)
 	(wire
@@
 					(unit 1)
 				)
-			)
-		)
-	)
-	(symbol
-		(lib_id "power:+5V")
-		(at 254 35.56 270)
-		(unit 1)
-		(exclude_from_sim no)
-		(in_bom yes)
-		(on_board yes)
-		(dnp no)
-		(fields_autoplaced yes)
-		(property "Reference" "#PWR039"
-			(at 250.19 35.56 0)
-			(effects
-				(font
-					(size 1.27 1.27)
-				)
-				(hide yes)
-			)
-		)
-		(property "Value" "+5V"
-			(at 257.81 35.5599 90)
-			(effects
-				(font
-					(size 1.27 1.27)
-				)
-				(justify left)
-			)
-		)
-		(property "Footprint" ""
-			(at 254 35.56 0)
-			(effects
-				(font
-					(size 1.27 1.27)
-				)
-				(hide yes)
-			)
-		)
-		(property "Datasheet" ""
-			(at 254 35.56 0)
-			(effects
-				(font
-					(size 1.27 1.27)
-				)
-				(hide yes)
-			)
-		)
-		(property "Description" "Power symbol creates a global label with name \"+5V\""
-			(at 254 35.56 0)
-			(effects
-				(font
-					(size 1.27 1.27)
-				)
-				(hide yes)
-			)
-		)
-		(pin "1"
-		)
-		(instances
-			(project ""
-				(path "/3e1046b6-e265-4cdd-8404-c358cfc105fe/0b285de8-9ee2-45ab-8a02-21d3047a383b"
-					(reference "#PWR039")
-					(unit 1)
-				)

Commit message: Fixes
Connections:
- net +5V: now also U5.J12_4 (+5V0), U5.J13_4 (+5V0), U5.J3_21 (+5V0), U5.JP5_1 (+5V0), U5.JP7_1 (+5V0)
- no-connect marks 1 -> 0
Changed lines of the file:
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@@
 		)
-	)
-	(no_connect
-		(at 254 35.56)
 	)
 	(wire
@@
 	(wire
 		(pts
-			(xy 30.48 41.91) (xy 33.02 41.91)
+			(xy 30.48 44.45) (xy 33.02 44.45)
 		)
 		(stroke
@@
 	(wire
 		(pts
+			(xy 254 35.56) (xy 250.19 35.56)
+		)
+		(stroke
+			(width 0)
+			(type default)
+		)
+	)
+	(wire
+		(pts
 			(xy 172.72 91.44) (xy 161.29 91.44)
 		)
@@
 	(wire
 		(pts
-			(xy 31.75 45.72) (xy 30.48 45.72)
+			(xy 31.75 48.26) (xy 30.48 48.26)
 		)
 		(stroke
@@
 		(pts
 			(xy 30.48 74.93) (xy 35.56 74.93)
-		)
-		(stroke
-			(width 0)
-			(type default)
-		)
-	)
-	(wire
-		(pts
-			(xy 254 35.56) (xy 250.19 35.56)
 		)
 		(stroke
@@
 	(hierarchical_label "+3.3VDC"
 		(shape input)
-		(at 30.48 45.72 180)
+		(at 30.48 48.26 180)
 		(effects
 			(font
@@
 	(hierarchical_label "GND"
 		(shape input)
-		(at 30.48 41.91 180)
+		(at 30.48 44.45 180)
 		(effects
 			(font
@@
 	(symbol
 		(lib_id "power:GND")
-		(at 33.02 41.91 90)
+		(at 33.02 44.45 90)
 		(unit 1)
 		(exclude_from_sim no)
@@
 		(fields_autoplaced yes)
 		(property "Reference" "#PWR038"
-			(at 39.37 41.91 0)
+			(at 39.37 44.45 0)
 			(effects
 				(font
@@
 		)
 		(property "Value" "GND"
-			(at 36.83 41.9101 90)
+			(at 36.83 44.4501 90)
 			(effects
 				(font
@@
 		)
 		(property "Footprint" ""
-			(at 33.02 41.91 0)
+			(at 33.02 44.45 0)
 			(effects
 				(font
@@
 		)
 		(property "Datasheet" ""
-			(at 33.02 41.91 0)
+			(at 33.02 44.45 0)
 			(effects
 				(font
@@
 		)
 		(property "Description" "Power symbol creates a global label with name \"GND\" , ground"
-			(at 33.02 41.91 0)
+			(at 33.02 44.45 0)
 			(effects
 				(font
@@
 				(path "/3e1046b6-e265-4cdd-8404-c358cfc105fe/0b285de8-9ee2-45ab-8a02-21d3047a383b"
 					(reference "#PWR038")
+					(unit 1)
+				)
+			)
+		)
+	)
+	(symbol
+		(lib_id "power:+5V")
+		(at 254 35.56 270)
+		(unit 1)
+		(exclude_from_sim no)
+		(in_bom yes)
+		(on_board yes)
+		(dnp no)
+		(fields_autoplaced yes)
+		(property "Reference" "#PWR093"
+			(at 250.19 35.56 0)
+			(effects
+				(font
+					(size 1.27 1.27)
+				)
+				(hide yes)
+			)
+		)
+		(property "Value" "+5V"
+			(at 257.81 35.5599 90)
+			(effects
+				(font
+					(size 1.27 1.27)
+				)
+				(justify left)
+			)
+		)
+		(property "Footprint" ""
+			(at 254 35.56 0)
+			(effects
+				(font
+					(size 1.27 1.27)
+				)
+				(hide yes)
+			)
+		)
+		(property "Datasheet" ""
+			(at 254 35.56 0)
+			(effects
+				(font
+					(size 1.27 1.27)
+				)
+				(hide yes)
+			)
+		)
+		(property "Description" "Power symbol creates a global label with name \"+5V\""
+			(at 254 35.56 0)
+			(effects
+				(font
+					(size 1.27 1.27)
+				)
+				(hide yes)
+			)
+		)
+		(pin "1"
+		)
+		(instances
+			(project "Custom Inverter PCB"
+				(path "/3e1046b6-e265-4cdd-8404-c358cfc105fe/0b285de8-9ee2-45ab-8a02-21d3047a383b"
+					(reference "#PWR093")
 					(unit 1)
 				)
@@
 	(symbol
 		(lib_id "power:+3.3V")
-		(at 31.75 45.72 270)
+		(at 31.75 48.26 270)
 		(unit 1)
 		(exclude_from_sim no)
@@
 		(fields_autoplaced yes)
 		(property "Reference" "#PWR037"
-			(at 27.94 45.72 0)
+			(at 27.94 48.26 0)
 			(effects
 				(font
@@
 		)
 		(property "Value" "+3.3VDC"
-			(at 35.56 45.7201 90)
+			(at 35.56 48.2601 90)
 			(effects
 				(font
@@
 		)
 		(property "Footprint" ""
-			(at 31.75 45.72 0)
+			(at 31.75 48.26 0)
 			(effects
 				(font
@@
 		)
 		(property "Datasheet" ""
-			(at 31.75 45.72 0)
+			(at 31.75 48.26 0)
 			(effects
 				(font
@@
 		)
 		(property "Description" "Power symbol creates a global label with name \"+3.3V\""
-			(at 31.75 45.72 0)
-			(effects
-				(font
+			(at 31.75 48.26 0)
+			(effects
+				(font

Commit message: PCB V3 changes
-HV outputs and inputs changed to screw terminals for lugs
- Fuses changes to 50A
- ADC pin for temp sense along with the temp sensing circuit
- Added more pins to motor encoder term for temp sense
Connections:
- net +3.3V: now also U5.J5_41 (J5_+3.3V)
- net ISENA: now also U5.J3_23 (ADCINA5); no longer U5.J7_67 (ADCINC3_P4I)
- net ISENB: now also U5.J3_24 (ADCINB0); no longer U5.J7_68 (ADCINC5_P6I)
- net ISENC: now also U5.J3_25 (ADCINC2); no longer U5.J7_69 (ADCINA3_P21)
- net Temp+: now reaches U5.J3_26 (ADCINB1)
- net +5V: no longer names the net of U5.J12_4 (+5V0), U5.J13_4 (+5V0), U5.J3_21 (+5V0), U5.JP5_1 (+5V0), U5.JP7_1 (+5V0)
Changed lines of the file:
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@@
+	(wire
+		(pts
+			(xy 30.48 36.83) (xy 40.64 36.83)
+		)
+		(stroke
+			(width 0)
+			(type default)
+		)
+	)
 	(wire
 		(pts
@@
 	(wire
 		(pts
-			(xy 33.02 71.12) (xy 35.56 71.12)
-		)
-		(stroke
-			(width 0)
-			(type default)
-		)
-	)
-	(wire
-		(pts
 			(xy 30.48 34.29) (xy 40.64 34.29)
 		)
@@
 	(wire
 		(pts
-			(xy 172.72 99.06) (xy 161.29 99.06)
-		)
-		(stroke
-			(width 0)
-			(type default)
-		)
-	)
-	(wire
-		(pts
 			(xy 101.6 114.3) (xy 110.49 114.3)
 		)
@@
 	(wire
 		(pts
+			(xy 106.68 81.28) (xy 110.49 81.28)
+		)
+		(stroke
+			(width 0)
+			(type default)
+		)
+	)
+	(wire
+		(pts
 			(xy 185.42 35.56) (xy 189.23 35.56)
 		)
@@
 	(wire
 		(pts
+			(xy 161.29 33.02) (xy 170.18 33.02)
+		)
+		(stroke
+			(width 0)
+			(type default)
+		)
+	)
+	(wire
+		(pts
 			(xy 250.19 71.12) (xy 254 71.12)
 		)
@@
 	(wire
 		(pts
-			(xy 172.72 96.52) (xy 161.29 96.52)
-		)
-		(stroke
-			(width 0)
-			(type default)
-		)
-	)
-	(wire
-		(pts
-			(xy 254 35.56) (xy 250.19 35.56)
-		)
-		(stroke
-			(width 0)
-			(type default)
-		)
-	)
-	(wire
-		(pts
 			(xy 172.72 91.44) (xy 161.29 91.44)
 		)
@@
 	(wire
 		(pts
-			(xy 161.29 93.98) (xy 172.72 93.98)
+			(xy 161.29 38.1) (xy 170.18 38.1)
 		)
 		(stroke
@@
 		(pts
 			(xy 30.48 80.01) (xy 35.56 80.01)
+		)
+		(stroke
+			(width 0)
+			(type default)
+		)
+	)
+	(wire
+		(pts
+			(xy 161.29 35.56) (xy 170.18 35.56)
+		)
+		(stroke
+			(width 0)
+			(type default)
+		)
+	)
+	(wire
+		(pts
+			(xy 161.29 30.48) (xy 170.18 30.48)
 		)
 		(stroke
@@
 		)
 	)
+	(label "TEMP+"
+		(at 40.64 36.83 180)
+		(effects
+			(font
+				(size 1.27 1.27)
+			)
+			(justify right bottom)
+		)
+	)
 	(label "SINE"
 		(at 172.72 83.82 180)
@@
 	)
 	(label "ISENB"
-		(at 172.72 96.52 180)
+		(at 170.18 33.02 180)
+		(effects
+			(font
+				(size 1.27 1.27)
+			)
+			(justify right bottom)
+		)
+	)
+	(label "TEMP+"
+		(at 170.18 38.1 180)
 		(effects
 			(font
@@
 	)
 	(label "ISENA"
-		(at 172.72 93.98 180)
+		(at 170.18 30.48 180)
 		(effects
 			(font
@@
 	)
 	(label "ISENC"
-		(at 172.72 99.06 180)
+		(at 170.18 35.56 180)
 		(effects
 			(font
@@
 		)
 	)
-	(hierarchical_label "+5V"
-		(shape output)
-		(at 35.56 71.12 0)
-		(effects
-			(font
-				(size 1.27 1.27)
-			)
-			(justify left)
+	(hierarchical_label "Temp+"
+		(shape input)
+		(at 30.48 36.83 180)
+		(effects
+			(font
+				(size 1.27 1.27)
+			)
+			(justify right)
 		)
 	)
@@
 	)
 	(symbol
-		(lib_id "power:+5V")
-		(at 254 35.56 270)
-		(unit 1)
-		(exclude_from_sim no)
-		(in_bom yes)
-		(on_board yes)
-		(dnp no)
-		(fields_autoplaced yes)
-		(property "Reference" "#PWR093"
-			(at 250.19 35.56 0)
-			(effects
-				(font
-					(size 1.27 1.27)
-				)
-				(hide yes)
-			)
-		)
-		(property "Value" "+5V"
-			(at 257.81 35.5599 90)
-			(effects
-				(font
-					(size 1.27 1.27)
-				)
-				(justify left)
-			)
-		)
-		(property "Footprint" ""
-			(at 254 35.56 0)
-			(effects
-				(font
-					(size 1.27 1.27)
-				)
-				(hide yes)
-			)
-		)
-		(property "Datasheet" ""
-			(at 254 35.56 0)
-			(effects
-				(font
-					(size 1.27 1.27)
-				)
-				(hide yes)
-			)
-		)
-		(property "Description" "Power symbol creates a global label with name \"+5V\""
-			(at 254 35.56 0)
-			(effects
-				(font
-					(size 1.27 1.27)
-				)
-				(hide yes)
-			)
-		)
-		(pin "1"
-		)
-		(instances
-			(project "Custom Inverter PCB"
-				(path "/3e1046b6-e265-4cdd-8404-c358cfc105fe/0b285de8-9ee2-45ab-8a02-21d3047a383b"
-					(reference "#PWR093")
-					(unit 1)
-				)
-			)
-		)
-	)
-	(symbol
-		(lib_id "power:+5V")
-		(at 33.02 71.12 90)
-		(unit 1)
-		(exclude_from_sim no)
-		(in_bom yes)
-		(on_board yes)
-		(dnp no)
-		(fields_autoplaced yes)
-		(property "Reference" "#PWR045"
-			(at 36.83 71.12 0)
-			(effects
-				(font
-					(size 1.27 1.27)
-				)
-				(hide yes)
-			)
-		)
-		(property "Value" "+5V"
-			(at 29.21 71.1199 90)
-			(effects
-				(font
-					(size 1.27 1.27)
-				)
-				(justify left)
-			)
-		)
-		(property "Footprint" ""
-			(at 33.02 71.12 0)
-			(effects
-				(font
-					(size 1.27 1.27)
-				)
-				(hide yes)
-			)
-		)
-		(property "Datasheet" ""
-			(at 33.02 71.12 0)
-			(effects
-				(font
-					(size 1.27 1.27)
-				)
-				(hide yes)
-			)
-		)
-		(property "Description" "Power symbol creates a global label with name \"+5V\""
-			(at 33.02 71.12 0)
-			(effects
-				(font
-					(size 1.27 1.27)
-				)
-				(hide yes)
-			)
-		)
-		(pin "1"
-		)
-		(instances
-			(project "Custom Inverter PCB"
-				(path "/3e1046b6-e265-4cdd-8404-c358cfc105fe/0b285de8-9ee2-45ab-8a02-21d3047a383b"
-					(reference "#PWR045")
-					(unit 1)
-				)
-			)
-		)
-	)
-	(symbol
 		(lib_id "10897202:10897202")
 		(at 217.17 105.41 0)
@@
 					(unit 1)
 				)
+			)
+		)
+	)
+	(symbol
+		(lib_id "power:+3.3V")
+		(at 106.68 81.28 90)
+		(mirror x)
+		(unit 1)
+		(exclude_from_sim no)
+		(in_bom yes)
+		(on_board yes)
+		(dnp no)
+		(property "Reference" "#PWR045"
+			(at 110.49 81.28 0)
+			(effects
+				(font
+					(size 1.27 1.27)
+				)
+				(hide yes)
+			)
+		)
+		(property "Value" "+3.3V"
+			(at 101.6 81.28 0)
+			(effects
+				(font
+					(size 1.27 1.27)
+				)
+			)
+		)
+		(property "Footprint" ""
+			(at 106.68 81.28 0)
+			(effects
+				(font
+					(size 1.27 1.27)
+				)
+				(hide yes)
+			)
+		)
+		(property "Datasheet" ""
+			(at 106.68 81.28 0)
+			(effects
+				(font
+					(size 1.27 1.27)
+				)
+				(hide yes)
+			)
+		)
+		(property "Description" "Power symbol creates a global label with name \"+3.3V\""
+			(at 106.68 81.28 0)
+			(effects
+				(font
+					(size 1.27 1.27)
+				)
+				(hide yes)
+			)
+		)
+		(pin "1"
+		)
+		(instances
+			(project "Custom Inverter PCB"
+				(path "/3e1046b6-e265-4cdd-8404-c358cfc105fe/0b285de8-9ee2-45ab-8a02-21d3047a383b"
+					(reference "#PWR045")
+					(unit 1)
+				)

Commit message: PCB layout
Parts:
- added C27: 220nF, Capacitor_SMD:C_0603_1608Metric, symbol Device:C
- renumbered J4 to J2, J5 to J3, J9 to J4, J10 to J5, U5 to U2
Connections:
- net GND: now also C27.2
- net Temp+: now also C27.1
- net OCD2_C: now reaches U2.J4_35 (GPIO5)
- net OCD1_C: now reaches U2.J4_36 (GPIO4)
- net OCD2_B: now reaches U2.J4_37 (GPIO9)
- net OCD1_B: now reaches U2.J4_38 (GPIO8)
- net OCD2_A: now reaches U2.J4_39 (GPIO11)
- net OCD1_A: now reaches U2.J4_40 (GPIO10)
