File: Power Hardware V3.0 (Live)/Custom Inverter PCB/_autosave-Encoder Input.kicad_sch (KiCad schematic)
At the start: 11 parts, among them J6 1989764, U6 OP292GSZ-REEL

Commit message: BOM list
Parts:
- removed C15: 0.1uF, Capacitor_SMD:C_0805_2012Metric, symbol Device:C
- removed J6: 1989764, PHOENIX_1989764:PHOENIX_1989764, symbol Connector:Conn_01x04_Socket
- added C17: 0.1uF, Capacitor_SMD:C_0805_2012Metric, symbol Device:C
- added J6: 1990041, PHOENIX_1990041:PHOENIX_1990041, symbol PHOENIX_1990041:1990041
- added R20: 5.36k, Resistor_SMD:R_0805_2012Metric, symbol Device:R
- renumbered R8 to R21, R45 to R22, R46 to R23, R5 to R24, R9 to R25, R48 to R26, R18 to R27, R47 to R28
Connections:
- net +5V: now also C17.1, J6.6, R20.2
- net COS_IN: now also J6.4
- net GND: now also C17.2, J6.1, J6.5
- net SIN_IN: now also J6.3
- new net TEMP+: J6.2, R20.1
Other:
- note added: "- Differential Opamp for subtracting some DC voltage from the Sin-Cos input"
- note added: "Connector To Motor"
- note removed: "-Changed 3.3V regulator to a higher power unit for the sin-cos circuit (from 500mA to 3A) -Fixed flipped MOTA,B,C connection to Output Terminal - Current Sense IC setup - Fuses for Phase current outputs - Differential Opamp for subtracting some DC voltage from the Sin-Cos input"
- note removed: "Connector To Resolver"
