File: Power Hardware V3.0 (Live)/Custom Inverter PCB/Current sense.kicad_sch (KiCad schematic)
At the start: 21 parts, among them U2 TLI4971A050T5E0001XUMA1, U3 TLI4971A050T5E0001XUMA1, U4 TLI4971A050T5E0001XUMA1

Commit message: Datasheets into components
Parts:
- U2: Part Number (none) -> TLI4971A050T5E0001XUMA1
Changed lines of the file:
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@@
 			)
 		)
-		(property "Datasheet" "TLI4971A050T5E0001XUMA1"
+		(property "Datasheet" "https://www.infineon.com/dgdl/Infineon-TLI4971_25_50_75_120-DataSheet-v01_20-EN.pdf?fileId=5546d462700c0ae6017034d731621b09"
 			(at 130.81 59.69 0)
 			(effects
@@
 			)
 		)
-		(property "Description" ""
+		(property "Description" "SENSOR CURRENT HALL 50A 8TISON"
 			(at 130.81 59.69 0)
 			(effects
@@
 			)
 		)
-		(property "Part Number" ""
+		(property "Part Number" "TLI4971A050T5E0001XUMA1"
 			(at 130.81 59.69 0)
 			(effects
@@
 			)
 		)
-		(property "Datasheet" "TLI4971A050T5E0001XUMA1"
+		(property "Datasheet" "https://www.infineon.com/dgdl/Infineon-TLI4971_25_50_75_120-DataSheet-v01_20-EN.pdf?fileId=5546d462700c0ae6017034d731621b09"
 			(at 132.08 87.63 0)
 			(effects
@@
 			)
 		)
-		(property "Description" ""
+		(property "Description" "SENSOR CURRENT HALL 50A 8TISON"
 			(at 132.08 87.63 0)
 			(effects
@@
 			)
 		)
-		(property "Datasheet" "TLI4971A050T5E0001XUMA1"
+		(property "Datasheet" "https://www.infineon.com/dgdl/Infineon-TLI4971_25_50_75_120-DataSheet-v01_20-EN.pdf?fileId=5546d462700c0ae6017034d731621b09"
 			(at 133.35 114.3 0)
 			(effects
@@
 			)
 		)
-		(property "Description" ""
+		(property "Description" "SENSOR CURRENT HALL 50A 8TISON"
 			(at 133.35 114.3 0)
 			(effects

Commit message: PCB layout
Parts:
- U3: renamed from U2; footprint TLI4971A:IC_TLI4971A050T5UE0001XUMA1 -> TLI4971A:TLI4971A050T5UE0001XUMA1
- U4: renamed from U3; footprint TLI4971A:IC_TLI4971A050T5UE0001XUMA1 -> TLI4971A:TLI4971A050T5UE0001XUMA1
- U5: renamed from U4; footprint TLI4971A:IC_TLI4971A050T5UE0001XUMA1 -> TLI4971A:TLI4971A050T5UE0001XUMA1
- renumbered C12 to C10, C13 to C12, C14 to C13, C24 to C14, C23 to C15, C21 to C16, R13 to R11, R14 to R12, R16 to R13, R12 to R14, R17 to R16, R32 to R17, R35 to R18, R36 to R19, R11 to R9

Commit message: V3.0 is ordered
Connections:
- net +3.3V renamed +3.3VDC

Commit message: changes
Parts:
- U4, U5: Part Number (none) -> TLI4971A050T5E0001XUMA1
Changed lines of the file:
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@@
 			)
 		)
-		(property "Part Number" ""
+		(property "Part Number" "TLI4971A050T5E0001XUMA1"
 			(at 132.08 87.63 0)
 			(effects
@@
 			)
 		)
-		(property "Part Number" ""
+		(property "Part Number" "TLI4971A050T5E0001XUMA1"
 			(at 133.35 114.3 0)
 			(effects
