File: Power Hardware V2.1/Custom Inverter PCB/Current sense.kicad_sch (KiCad schematic)
At the start: 21 parts, among them U2 TLI4971A050T5E0001XUMA1, U3 TLI4971A050T5E0001XUMA1, U4 TLI4971A050T5E0001XUMA1

Commit message: BOM list
Parts:
- U2, U3, U4: Part Number (none) -> TLI4971A050T5E0001XUMA1
Changed lines of the file:
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@@
 			)
 		)
-		(property "Part Number" ""
+		(property "Part Number" "TLI4971A050T5E0001XUMA1"
 			(at 130.81 59.69 0)
 			(effects
@@
 			)
 		)
-		(property "Part Number" ""
+		(property "Part Number" "TLI4971A050T5E0001XUMA1"
 			(at 132.08 87.63 0)
 			(effects
@@
 			)
 		)
-		(property "Part Number" ""
+		(property "Part Number" "TLI4971A050T5E0001XUMA1"
 			(at 133.35 114.3 0)
 			(effects
