File: Power Hardware V2.1/Custom Inverter PCB/Gate_Driver_PowerInputs.kicad_sch (KiCad schematic)
At the start: 22 parts, among them J1 1714971, J2 1714971, J3 1714968, J7 1714971, J8 1714971, K2 1-1393210-3, U1 DRV8300DIPWR

Commit message: BOM list
Parts:
- CR4: Part Number (none) -> LD1085D2M33R
- F1: Part Number (none) -> 0463030.ER
- J1, J2, J7, J8: Part Number (none) -> 1714971
- J3: Part Number (none) -> 1714968
- K2: Part Number (none) -> T9AS1D12-12
- U1: Part Number (none) -> DRV8300DIPWR
Changed lines of the file:
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@@
 			)
 		)
-		(property "Part Number" ""
+		(property "Part Number" "DRV8300DIPWR"
 			(at 173.99 30.48 0)
 			(effects
@@
 			)
 		)
-		(property "Part Number" ""
+		(property "Part Number" "0463030.ER"
 			(at 64.77 22.86 0)
 			(effects
@@
 			)
 		)
+		(property "Part Number" "1714971"
+			(at 26.67 59.69 0)
+			(effects
+				(font
+					(size 1.27 1.27)
+				)
+				(hide yes)
+			)
+		)
 		(pin "1"
 		)
@@
 			)
 		)
-		(property "Part Number" ""
+		(property "Part Number" "1714968"
 			(at 265.43 90.17 0)
 			(effects
@@
 			)
 		)
-		(property "Datasheet" "LD1085D2M33R"
+		(property "Datasheet" ""
 			(at 133.35 147.32 0)
 			(effects
@@
 			)
 		)
+		(property "Part Number" "LD1085D2M33R"
+			(at 133.35 147.32 0)
+			(effects
+				(font
+					(size 1.27 1.27)
+				)
+				(hide yes)
+			)
+		)
 		(pin "4"
 		)
@@
 			)
 		)
+		(property "Part Number" "1714971"
+			(at 82.55 116.84 90)
+			(effects
+				(font
+					(size 1.27 1.27)
+				)
+				(hide yes)
+			)
+		)
 		(pin "2"
 		)
@@
 			)
 		)
-		(property "Part Number" ""
+		(property "Part Number" "T9AS1D12-12"
 			(at 123.19 67.31 0)
 			(effects
@@
 			)
 		)
+		(property "Part Number" "1714971"
+			(at 85.09 78.74 90)
+			(effects
+				(font
+					(size 1.27 1.27)
+				)
+				(hide yes)
+			)
+		)
 		(pin "2"
 		)
@@
 				(hide yes)
 			)
+		)
+		(property "Part Number" "1714971"
+			(at 26.67 29.21 0)
+			(effects
+				(font
+					(size 1.27 1.27)
+				)
+				(hide yes)
+			)
