File: Power Hardware V2.1/Custom Inverter PCB/Half_Bridges.kicad_sch (KiCad schematic)
At the start: 27 parts, among them Q1 CSD19532Q5B, Q2 CSD19532Q5B, Q3 CSD19532Q5B, Q4 CSD19532Q5B, Q5 CSD19532Q5B, Q6 CSD19532Q5B

Commit message: BOM list
Parts:
- Q1, Q2, Q3, Q4, Q5, Q6: Part Number (none) -> CSD19532Q5B
- TP1, TP2, TP3, TP4, TP5, TP6, TP7, TP8, TP9: Part Number (none) -> 5002
Changed lines of the file:
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@@
 			)
 		)
-		(property "Part Number" ""
+		(property "Part Number" "5002"
 			(at 274.32 57.15 0)
 			(effects
@@
 			)
 		)
-		(property "Part Number" ""
+		(property "Part Number" "5002"
 			(at 92.71 57.15 0)
 			(effects
@@
 			)
 		)
-		(property "Part Number" ""
+		(property "Part Number" "5002"
 			(at 30.48 73.66 0)
 			(effects
@@
 			)
 		)
-		(property "Part Number" ""
+		(property "Part Number" "CSD19532Q5B"
 			(at 55.88 76.2 0)
 			(effects
@@
 			)
 		)
-		(property "Part Number" ""
+		(property "Part Number" "5002"
 			(at 209.55 46.99 0)
 			(effects
@@
 			)
 		)
-		(property "Part Number" ""
+		(property "Part Number" "CSD19532Q5B"
 			(at 229.87 49.53 0)
 			(effects
@@
 			)
 		)
-		(property "Part Number" ""
+		(property "Part Number" "5002"
 			(at 29.21 46.99 0)
 			(effects
@@
 			)
 		)
-		(property "Part Number" ""
+		(property "Part Number" "CSD19532Q5B"
 			(at 229.87 76.2 0)
 			(effects
@@
 			)
 		)
-		(property "Part Number" ""
+		(property "Part Number" "CSD19532Q5B"
 			(at 55.88 49.53 0)
 			(effects
@@
 			)
 		)
-		(property "Part Number" ""
+		(property "Part Number" "5002"
 			(at 121.92 73.66 0)
 			(effects
@@
 			)
 		)
-		(property "Part Number" ""
+		(property "Part Number" "CSD19532Q5B"
 			(at 143.51 76.2 0)
 			(effects
@@
 			)
 		)
-		(property "Part Number" ""
+		(property "Part Number" "5002"
 			(at 181.61 57.15 0)
 			(effects
@@
 			)
 		)
-		(property "Part Number" ""
+		(property "Part Number" "5002"
 			(at 210.82 73.66 0)
 			(effects
@@
 			)
 		)
-		(property "Part Number" ""
+		(property "Part Number" "5002"
 			(at 120.65 46.99 0)
 			(effects
@@
 			)
 		)
-		(property "Part Number" ""
+		(property "Part Number" "CSD19532Q5B"
 			(at 143.51 49.53 0)
 			(effects
