File: Power Hardware V2.1/Custom Inverter PCB/MCU.kicad_sch (KiCad schematic)
At the start: 5 parts, among them J10 10897202, J4 10897202, J5 10897202, J9 10897202, U5 LAUNCHXL-F280049C

Commit message: BOM list
Parts:
- J10, J4, J5, J9: Part Number (none) -> 10897202
- U5: Part Number (none) -> LAUNCHXL-F280049C
Changed lines of the file:
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@@
+			)
+		)
+		(property "Part Number" "10897202"
+			(at 217.17 105.41 90)
+			(effects
+				(font
+					(size 1.27 1.27)
+				)
+				(hide yes)
 			)
 		)
@@
 			)
 		)
-		(property "Part Number" ""
+		(property "Part Number" "LAUNCHXL-F280049C"
 			(at 135.89 78.74 0)
 			(effects
@@
 		(property "Description" ""
 			(at 196.85 105.41 0)
+			(effects
+				(font
+					(size 1.27 1.27)
+				)
+				(hide yes)
+			)
+		)
+		(property "Part Number" "10897202"
+			(at 196.85 105.41 90)
 			(effects
 				(font
@@
 			)
 		)
+		(property "Part Number" "10897202"
+			(at 257.81 105.41 0)
+			(effects
+				(font
+					(size 1.27 1.27)
+				)
+				(hide yes)
+			)
+		)
 		(pin "7"
 		)
@@
 			)
 		)
-		(property "Part Number" ""
+		(property "Part Number" "LAUNCHXL-F280049C"
 			(at 219.71 55.88 0)
 			(effects
@@
 			(at 236.22 105.41 0)
 			(effects
+				(font
+					(size 1.27 1.27)
+				)
+				(hide yes)
+			)
+		)
+		(property "Part Number" "10897202"
+			(at 236.22 105.41 0)
+			(effects
